File: beeper/beeper.sch (KiCad schematic (older format))
At the start: 30 parts, among them J1 Conn_01x03, J2 TEST_1P, J3 TEST_1P, J4 TEST_1P, J5 TEST_1P, Q2 Q_NMOS_DGS, SW1 SW_Push, U1 ATTINY13A-SSU, U2 MCP73831-2-OT

Commit message: Version 2.
Parts:
- BT1: footprint Pin_Headers:Pin_Header_Straight_2x01_Pitch2.54mm -> Connector_PinHeader_1.00mm:PinHeader_2x01_P1.00mm_Vertical_SMD; symbol Battery_Cell_switched -> my_components:Battery_Cell_switched
- BZ1: footprint Buzzers_Beepers:BUZZER -> Buzzer_Beeper:Buzzer_12x9.5RM7.6; symbol Buzzer -> beeper-rescue:Buzzer
- C1, C4: footprint Capacitors_SMD:C_0805 -> Capacitor_SMD:C_0805_2012Metric; symbol C -> pspice:C
- C2, C3: footprint Capacitors_SMD:C_0603 -> Capacitor_SMD:C_0603_1608Metric; symbol C -> pspice:C
- D1, D2: footprint LEDs:LED_0805 -> LED_SMD:LED_0805_2012Metric_Castellated; symbol LED -> beeper-rescue:LED
- J1: footprint Pin_Headers:Pin_Header_Straight_1x03_Pitch2.54mm -> Connector_PinHeader_2.54mm:PinHeader_1x03_P2.54mm_Vertical; symbol Conn_01x03 -> beeper-rescue:Conn_01x03
- J2, J3, J4, J5: footprint Measurement_Points:Measurement_Point_Round-SMD-Pad_Small -> TestPoint:TestPoint_Pad_D1.0mm; symbol TEST_1P -> beeper-rescue:TEST_1P
- JP1, JP2: footprint (none) -> Jumper:SolderJumper-3_P1.3mm_Open_RoundedPad1.0x1.5mm; symbol Jumper_NC_Dual -> beeper-rescue:Jumper_NC_Dual
- MK1, MK2: footprint Mounting_Holes:MountingHole_3.2mm_M3 -> MountingHole:MountingHole_3.2mm_M3; symbol Mounting_Hole -> beeper-rescue:Mounting_Hole
- Q2: footprint TO_SOT_Packages_SMD:SOT-23 -> Package_TO_SOT_SMD:SOT-23; symbol Q_NMOS_GSD -> beeper-rescue:Q_NMOS_GSD
- R1, R2, R3, R4, R5, R6, R7, R8, R9: footprint Resistors_SMD:R_0805 -> Resistor_SMD:R_0805_2012Metric; symbol R -> pspice:R
- SW1: footprint Buttons_Switches_SMD:SW_DIP_x1_W5.08mm_Slide_Copal_CHS-A -> Button_Switch_SMD:SW_SPST_CK_RS282G05A3; symbol SW_Push -> beeper-rescue:SW_Push
- U1: footprint Housings_SOIC:SOIC-8_3.9x4.9mm_Pitch1.27mm -> Package_SO:SOIC-8_3.9x4.9mm_P1.27mm; symbol ATTINY13A-SSU -> beeper-rescue:ATTINY13A-SSU
- U2: footprint TO_SOT_Packages_SMD:SOT-23-5 -> Package_TO_SOT_SMD:SOT-23-5; symbol MCP73831-2-OT -> beeper-rescue:MCP73831-2-OT

Commit message: PCB v0.2
Parts:
- removed JP1, JP2: Jumper_NC_Dual, Jumper:SolderJumper-3_P1.3mm_Open_RoundedPad1.0x1.5mm, symbol beeper-rescue:Jumper_NC_Dual
- added BZ2: Buzzer, Buzzer_Beeper:Buzzer_Murata_PKMCS0909E4000-R1, symbol beeper-rescue:Buzzer
- added D3: D, Diode_SMD:D_0805_2012Metric, symbol Device:D
- BT1: footprint Connector_PinHeader_1.00mm:PinHeader_2x01_P1.00mm_Vertical_SMD -> Connector_PinHeader_2.00mm:PinHeader_2x01_P2.00mm_Vertical
- J2: value TEST_1P -> SCK
- J3: value TEST_1P -> MISO
- J4: value TEST_1P -> RST
- J5: value TEST_1P -> MOSI
- Q2: value Q_NMOS_DGS -> irlml2502
- R4: value 100k -> 10k
Connections:
- net BUZZER_GND: now also BZ1.2 (+), Q2.3 (D), BZ2.2 (+), D3.2 (A); no longer Q2.2 (S)
- net BUZZER_OUT: now also J5.1, U1.5 (PB0(MOSI/AIN0/OC0A/PCINT0)); no longer U1.2 (PB3(CLKI/ADC3/PCINT3))
- net Beeper_in: now also U1.2 (PB3(CLKI/ADC3/PCINT3)); no longer J2.1, U1.5 (PB0(MOSI/AIN0/OC0A/PCINT0))
- net GND: now also Q2.2 (S); no longer Q2.3 (D)
- net STATUS_OUT: now also J2.1; no longer J5.1
- net VCC: now also BZ1.1 (-), BZ2.1 (-), D3.1 (K)
- net at C3.2, R7.2, U1.1 (PB5(~RESET~/ADC0/PCINT5/dW)): now also J4.1; no longer J3.1
- net at SW1.2, U1.6 (PB1(MISO/AIN1/OC0B/INT0/PCINT1)): now also J3.1; no longer J4.1
Other:
- note added: "Buzzer with diode\n"
- note added: "Pulldown since the avr \ncan only do pullup"
- note removed: "Buzzer polarity selection\n"
- moved on the sheet: BZ1
Changed lines of the file:
@@
 	1    0    0    -1
 $EndComp
-Text Label 2950 3700 0    60   ~ 0
+Text Label 2900 4000 0    60   ~ 0
 Beeper_in
 $Comp
@@
 L beeper-rescue:Buzzer BZ1
 U 1 1 5C3D137A
-P 5050 2750
-F 0 "BZ1" H 5200 2800 50  0000 L CNN
-F 1 "Buzzer" H 5200 2700 50  0000 L CNN
-F 2 "Buzzer_Beeper:Buzzer_12x9.5RM7.6" V 5025 2850 50  0001 C CNN
-F 3 "" V 5025 2850 50  0001 C CNN
-	1    5050 2750
+P 5700 2750
+F 0 "BZ1" H 5850 2800 50  0000 L CNN
+F 1 "Buzzer" H 5850 2700 50  0000 L CNN
+F 2 "Buzzer_Beeper:Buzzer_12x9.5RM7.6" V 5675 2850 50  0001 C CNN
+F 3 "" V 5675 2850 50  0001 C CNN
+	1    5700 2750
 	1    0    0    -1
 $EndComp
@@
 P 2600 1350
 F 0 "Q2" H 2800 1400 50  0000 L CNN
-F 1 "Q_NMOS_DGS" H 2800 1300 50  0000 L CNN
+F 1 "irlml2502" H 2800 1300 50  0000 L CNN
 F 2 "Package_TO_SOT_SMD:SOT-23" H 2800 1450 50  0001 C CNN
 F 3 "" H 2600 1350 50  0001 C CNN
 	1    2600 1350
-	-1   0    0    1
+	-1   0    0    -1
 $EndComp
 $Comp
@@
 P 2850 1650
 F 0 "R4" V 2930 1650 50  0000 C CNN
-F 1 "100k" V 2850 1650 50  0000 C CNN
+F 1 "10k" V 2850 1650 50  0000 C CNN
 F 2 "Resistor_SMD:R_0805_2012Metric" H 2850 1650 50  0001 C CNN
 F 3 "" H 2850 1650 50  0001 C CNN
@@
 F 3 "" H 2500 1950 50  0001 C CNN
 	1    2500 1950
-	1    0    0    -1
-$EndComp
-$Comp
-L beeper-rescue:TEST_1P J3
-U 1 1 5C3E3019
-P 3450 5050
-F 0 "J3" H 3450 5320 50  0000 C CNN
-F 1 "TEST_1P" H 3450 5250 50  0000 C CNN
-F 2 "TestPoint:TestPoint_Pad_D1.0mm" H 3650 5050 50  0001 C CNN
-F 3 "" H 3650 5050 50  0001 C CNN
-	1    3450 5050
-	-1   0    0    1
-$EndComp
-$Comp
-L beeper-rescue:TEST_1P J2
-U 1 1 5C3E319D
-P 3400 3600
-F 0 "J2" H 3400 3870 50  0000 C CNN
-F 1 "TEST_1P" H 3400 3800 50  0000 C CNN
-F 2 "TestPoint:TestPoint_Pad_D1.0mm" H 3600 3600 50  0001 C CNN
-F 3 "" H 3600 3600 50  0001 C CNN
-	1    3400 3600
-	1    0    0    -1
-$EndComp
-$Comp
-L beeper-rescue:TEST_1P J5
-U 1 1 5C3E375D
-P 900 4400
-F 0 "J5" H 900 4670 50  0000 C CNN
-F 1 "TEST_1P" H 900 4600 50  0000 C CNN
-F 2 "TestPoint:TestPoint_Pad_D1.0mm" H 1100 4400 50  0001 C CNN
-F 3 "" H 1100 4400 50  0001 C CNN
-	1    900  4400
-	0    -1   -1   0
-$EndComp
-$Comp
-L beeper-rescue:TEST_1P J4
-U 1 1 5C3E395C
-P 2800 3600
-F 0 "J4" H 2800 3870 50  0000 C CNN
-F 1 "TEST_1P" H 2800 3800 50  0000 C CNN
-F 2 "TestPoint:TestPoint_Pad_D1.0mm" H 3000 3600 50  0001 C CNN
-F 3 "" H 3000 3600 50  0001 C CNN
-	1    2800 3600
 	1    0    0    -1
 $EndComp
@@
 Text Notes 800  1350 0    60   ~ 0
 Input from FC
-Text Label 2900 4000 0    60   ~ 0
+Text Label 2950 3700 0    60   ~ 0
 BUZZER_OUT
 Text Label 3500 750  2    60   ~ 0
@@
 	2950 750  3500 750
 Wire Wire Line
-	2950 3700 3400 3700
-Wire Wire Line
 	500  2300 1100 2300
 Wire Wire Line
@@
 Connection ~ 2800 2800
 Wire Wire Line
-	2750 3800 2800 3800
-Wire Wire Line
 	5450 4200 5600 4200
 Wire Wire Line
@@
 	2300 3800 2350 3800
 Wire Wire Line
-	2800 3600 2800 3800
-Connection ~ 2800 3800
-Wire Wire Line
-	3400 3700 3400 3600
-Connection ~ 3400 3700
-Wire Wire Line
 	1100 1550 1100 1650
 Wire Wire Line
@@
 Wire Wire Line
 	3450 4750 3500 4750
-Connection ~ 3450 4750
 Wire Wire Line
 	4000 4750 4100 4750
@@
 Wire Wire Line
 	6850 1350 6800 1350
-Wire Wire Line
-	2950 3900 3450 3900
-Wire Wire Line
-	900  4400 1050 4400
 Wire Wire Line
 	1050 4400 1050 4450
@@
 Wire Notes Line
 	1800 5750 450  5750
-Connection ~ 1050 4400
 $Comp
 L my_components:Battery_Cell_switched BT1
@@
 F 0 "BT1" H 4500 1100 50  0000 L CNN
 F 1 "Battery_Cell_switched" H 3950 950 50  0000 L CNN
-F 2 "Connector_PinHeader_1.00mm:PinHeader_2x01_P1.00mm_Vertical_SMD" V 4400 1060 50  0001 C CNN
+F 2 "Connector_PinHeader_2.00mm:PinHeader_2x01_P2.00mm_Vertical" V 4400 1060 50  0001 C CNN
 F 3 "" V 4400 1060 50  0001 C CNN
 	1    4400 1000
@@
 L power:VCC #PWR025
 U 1 1 5C83D9E9
-P 4150 2700
-F 0 "#PWR025" H 4150 2550 50  0001 C CNN
-F 1 "VCC" H 4150 2850 50  0000 C CNN
-F 2 "" H 4150 2700 50  0001 C CNN
-F 3 "" H 4150 2700 50  0001 C CNN
-	1    4150 2700
-	0    -1   -1   0
-$EndComp
-$Comp
-L beeper-rescue:Jumper_NC_Dual JP1
-U 1 1 5C83E5B6
-P 4550 2400
-F 0 "JP1" H 4600 2300 50  0000 L CNN
-F 1 "Jumper_NC_Dual" H 4550 2500 50  0000 C BNN
-F 2 "Jumper:SolderJumper-3_P1.3mm_Open_RoundedPad1.0x1.5mm" H 4550 2400 50  0001 C CNN
-F 3 "" H 4550 2400 50  0001 C CNN
-	1    4550 2400
-	1    0    0    -1
-$EndComp
-Wire Wire Line
-	4950 2650 4550 2650
-Wire Wire Line
-	4550 2650 4550 2500
-Wire Wire Line
-	4800 2400 5600 2400
-$Comp
-L beeper-rescue:Jumper_NC_Dual JP2
-U 1 1 5C83EAE0
-P 4550 3000
-F 0 "JP2" H 4600 2900 50  0000 L CNN
-F 1 "Jumper_NC_Dual" H 4550 3100 50  0000 C BNN
-F 2 "Jumper:SolderJumper-3_P1.3mm_Open_RoundedPad1.0x1.5mm" H 4550 3000 50  0001 C CNN
-F 3 "" H 4550 3000 50  0001 C CNN
-	1    4550 3000
-	-1   0    0    1
-$EndComp
-Wire Wire Line
-	4550 2900 4550 2850
-Wire Wire Line
-	4550 2850 4950 2850
-Wire Wire Line
-	5600 3000 4800 3000
-Wire Wire Line
-	4300 2400 4250 2400
-Wire Wire Line
-	4250 2400 4250 2700
-Wire Wire Line
-	4250 3000 4300 3000
-Wire Wire Line
-	4150 2700 4250 2700
-Connection ~ 4250 2700
-Wire Wire Line
-	5600 2400 5600 2750
-Connection ~ 5600 2750
-Text Label 6200 2750 2    60   ~ 0
+P 4950 2600
+F 0 "#PWR025" H 4950 2450 50  0001 C CNN
+F 1 "VCC" H 4950 2750 50  0000 C CNN
+F 2 "" H 4950 2600 50  0001 C CNN
+F 3 "" H 4950 2600 50  0001 C CNN
+	1    4950 2600
+	0    -1   -1   0
+$EndComp
+Text Label 4450 2900 0    60   ~ 0
 BUZZER_GND
-Wire Wire Line
-	5600 2750 6200 2750
 Text Label 2500 550  3    60   ~ 0
 BUZZER_GND
 Text Notes 5500 2350 0    60   ~ 0
-Buzzer polarity selection\n
+Buzzer with diode\n
 Wire Notes Line
 	3850 3200 7200 3200
@@
 	2850 1350 2950 1350
 Wire Wire Line
-	2800 3800 3450 3800
+	1100 2300 1200 2300
+Wire Wire Line
+	3450 4400 3450 4750
+Wire Wire Line
+	5800 1900 5800 2000
+Wire Wire Line
+	5800 850  5800 950
+Wire Wire Line
+	5800 850  6550 850
+Wire Wire Line
+	1050 4400 1650 4400
+Wire Wire Line
+	2750 3800 2850 3800
+Wire Wire Line
+	2950 3700 3400 3700
+Text Notes 500  1650 0    50   ~ 0
+Pulldown since the avr \ncan only do pullup
+$Comp
+L beeper-rescue:TEST_1P J2
+U 1 1 5C84337F
+P 2650 4000
+F 0 "J2" H 2592 4027 50  0000 R CNN
+F 1 "SCK" H 2592 4118 50  0000 R CNN
+F 2 "TestPoint:TestPoint_Pad_D1.0mm" H 2850 4000 50  0001 C CNN
+F 3 "" H 2850 4000 50  0001 C CNN
+	1    2650 4000
+	-1   0    0    1
+$EndComp
+Wire Wire Line
+	2650 3900 2650 4000
+Wire Wire Line
+	2650 3900 3450 3900
+$Comp
+L beeper-rescue:TEST_1P J3
+U 1 1 5C84707B
+P 2850 3550
+F 0 "J3" H 2908 3670 50  0000 L CNN
+F 1 "MISO" H 2908 3579 50  0000 L CNN
+F 2 "TestPoint:TestPoint_Pad_D1.0mm" H 3050 3550 50  0001 C CNN
+F 3 "" H 3050 3550 50  0001 C CNN
+	1    2850 3550
+	1    0    0    -1
+$EndComp
+Wire Wire Line
+	2850 3550 2850 3800
+Connection ~ 2850 3800
+Wire Wire Line
+	2850 3800 3450 3800
+$Comp
+L beeper-rescue:TEST_1P J5
+U 1 1 5C848950
+P 3400 3500
+F 0 "J5" H 3458 3620 50  0000 L CNN
+F 1 "MOSI" H 3458 3529 50  0000 L CNN
+F 2 "TestPoint:TestPoint_Pad_D1.0mm" H 3600 3500 50  0001 C CNN
+F 3 "" H 3600 3500 50  0001 C CNN
+	1    3400 3500
+	1    0    0    -1
+$EndComp
+Wire Wire Line
+	3400 3500 3400 3700
+Connection ~ 3400 3700
 Wire Wire Line
 	3400 3700 3450 3700
-Wire Wire Line
-	1100 2300 1200 2300
-Wire Wire Line
-	3450 4400 3450 4750
-Wire Wire Line
-	3450 4750 3450 5050
-Wire Wire Line
-	5800 1900 5800 2000
-Wire Wire Line
-	5800 850  5800 950
-Wire Wire Line
-	5800 850  6550 850
-Wire Wire Line
-	1050 4400 1650 4400
-Wire Wire Line
-	4250 2700 4250 3000
-Wire Wire Line
-	5600 2750 5600 3000
+$Comp
+L beeper-rescue:TEST_1P J4
+U 1 1 5C84A91B
+P 3300 4750
+F 0 "J4" V 3495 4824 50  0000 C CNN
+F 1 "RST" V 3404 4824 50  0000 C CNN
+F 2 "TestPoint:TestPoint_Pad_D1.0mm" H 3500 4750 50  0001 C CNN
+F 3 "" H 3500 4750 50  0001 C CNN
+	1    3300 4750
+	0    -1   -1   0
+$EndComp
+Wire Wire Line
+	3300 4750 3450 4750
+Connection ~ 3450 4750
+$Comp
+L Device:D D3
+U 1 1 5CDA5B53
+P 5150 2750
+F 0 "D3" V 5104 2829 50  0000 L CNN
+F 1 "D" V 5195 2829 50  0000 L CNN
+F 2 "Diode_SMD:D_0805_2012Metric" H 5150 2750 50  0001 C CNN
+F 3 "~" H 5150 2750 50  0001 C CNN
+	1    5150 2750
+	0    1    1    0
+$EndComp
+Wire Wire Line
+	5150 2900 5600 2900
+Wire Wire Line
+	5600 2900 5600 2850
+Wire Wire Line
+	5150 2600 5600 2600
+Wire Wire Line
+	5600 2600 5600 2650
+Wire Wire Line
+	4950 2600 5150 2600
+Connection ~ 5150 2600
+Wire Wire Line
+	5150 2900 4450 2900
+Connection ~ 5150 2900
+$Comp
+L beeper-rescue:Buzzer BZ2
+U 1 1 5CDB2B4E
+P 6300 2750
+F 0 "BZ2" H 6450 2800 50  0000 L CNN
+F 1 "Buzzer" H 6450 2700 50  0000 L CNN
+F 2 "Buzzer_Beeper:Buzzer_Murata_PKMCS0909E4000-R1" V 6275 2850 50  0001 C CNN
+F 3 "" V 6275 2850 50  0001 C CNN
+	1    6300 2750
+	1    0    0    -1
+$EndComp
+Wire Wire Line
+	5600 2600 6200 2600
+Wire Wire Line
+	6200 2600 6200 2650
+Connection ~ 5600 2600
+Wire Wire Line
+	6200 2850 6200 2900
+Wire Wire Line
+	6200 2900 5600 2900
+Connection ~ 5600 2900
 $EndSCHEMATC

Commit message: PCB v0.2 final
Parts:
- added JP1: enable buzzer, Jumper:SolderJumper-2_P1.3mm_Open_RoundedPad1.0x1.5mm, symbol Device:Jumper_NO_Small
- BZ1: footprint Buzzer_Beeper:Buzzer_12x9.5RM7.6 -> buzzer:Buzzer_12x9.5RM7.6_oval3
Connections:
- net BUZZER_OUT: now also JP1.1; no longer J5.1, U1.5 (PB0(MOSI/AIN0/OC0A/PCINT0))
- new net: J5.1, JP1.2, U1.5 (PB0(MOSI/AIN0/OC0A/PCINT0))
Other:
- note added: "Remove this jumper for flashing"
Changed lines of the file:
@@
 EESchema Schematic File Version 4
 LIBS:beeper-cache
-EELAYER 26 0
+EELAYER 29 0
 EELAYER END
 $Descr A4 11693 8268
@@
 F 0 "BZ1" H 5850 2800 50  0000 L CNN
 F 1 "Buzzer" H 5850 2700 50  0000 L CNN
-F 2 "Buzzer_Beeper:Buzzer_12x9.5RM7.6" V 5675 2850 50  0001 C CNN
+F 2 "buzzer:Buzzer_12x9.5RM7.6_oval3" V 5675 2850 50  0001 C CNN
 F 3 "" V 5675 2850 50  0001 C CNN
 	1    5700 2750
@@
 Text Notes 800  1350 0    60   ~ 0
 Input from FC
-Text Label 2950 3700 0    60   ~ 0
+Text Label 1850 3700 0    60   ~ 0
 BUZZER_OUT
 Text Label 3500 750  2    60   ~ 0
@@
 Wire Wire Line
 	2750 3800 2850 3800
-Wire Wire Line
-	2950 3700 3400 3700
 Text Notes 500  1650 0    50   ~ 0
 Pulldown since the avr \ncan only do pullup
@@
 	6200 2900 5600 2900
 Connection ~ 5600 2900
+$Comp
+L Device:Jumper_NO_Small JP1
+U 1 1 5CE17746
+P 2300 3700
+F 0 "JP1" H 2250 4000 50  0000 C CNN
+F 1 "enable buzzer" H 2300 3850 50  0000 C CNN
+F 2 "Jumper:SolderJumper-2_P1.3mm_Open_RoundedPad1.0x1.5mm" H 2300 3700 50  0001 C CNN
+F 3 "~" H 2300 3700 50  0001 C CNN
+	1    2300 3700
+	1    0    0    -1
+$EndComp
+Text Notes 1900 3150 0    50   ~ 0
+Remove this jumper for flashing
+Wire Wire Line
+	1850 3700 2200 3700
+Wire Wire Line
+	2400 3700 3400 3700
 $EndSCHEMATC

Commit message: Final v0.2 (ordered)
Parts:
- D3: value D -> 1N4148; footprint Diode_SMD:D_0805_2012Metric -> Diode_SMD:D_SOD-323
Changed lines of the file:
@@
 P 5150 2750
 F 0 "D3" V 5104 2829 50  0000 L CNN
-F 1 "D" V 5195 2829 50  0000 L CNN
-F 2 "Diode_SMD:D_0805_2012Metric" H 5150 2750 50  0001 C CNN
+F 1 "1N4148" V 5195 2829 50  0000 L CNN
+F 2 "Diode_SMD:D_SOD-323" H 5150 2750 50  0001 C CNN
 F 3 "~" H 5150 2750 50  0001 C CNN
 	1    5150 2750
